Commit message: Add MoveIt pick cube functionality with improved gripper
- Added pick_cube_moveit_py.py:

File: kawada_repo-main/nextage_fillie_open_description/urdf/simple_gripper.xacro (robot description, xacro)
@@ -79,5 +79,5 @@
       <child link="${prefix}_gripper_left_finger"/>
       <axis xyz="0 1 0"/>
-      <limit lower="0.0" upper="0.04" effort="100" velocity="0.5"/>
+      <limit lower="0.0" upper="0.08" effort="100" velocity="0.5"/>
     </joint>
     <!-- Right Finger -->
@@ -130,5 +130,5 @@
       <child link="${prefix}_gripper_right_finger"/>
       <axis xyz="0 1 0"/>
-      <limit lower="-0.04" upper="0.0" effort="100" velocity="0.5"/>
+      <limit lower="-0.08" upper="0.0" effort="100" velocity="0.5"/>
       <mimic joint="${prefix}_gripper_left_finger_joint" multiplier="-1" offset="0"/>
     </joint>
