Commit message: Refine simple_pick approach

File: kawada_repo-main/kawada_moveit_config/config/NEXTAGE.ros2_control.xacro (robot description, xacro)
@@ -50,4 +50,11 @@
                 <state_interface name="velocity"/>
             </joint>
+            <joint name="right_gripper_left_finger_joint">
+                <command_interface name="position"/>
+                <state_interface name="position">
+                  <param name="initial_value">0.0</param>
+                </state_interface>
+                <state_interface name="velocity"/>
+            </joint>
         </ros2_control>
     </xacro:macro>

File: kawada_repo-main/kawada_moveit_config/config/NEXTAGE.urdf.xacro (robot description, xacro)
@@ -19,4 +19,6 @@
     <!-- Import cameras -->
     <xacro:include filename="$(find kawada_moveit_config)/config/cameras.xacro"/>
+    <!-- Import gripper -->
+    <xacro:include filename="$(find nextage_fillie_open_description)/urdf/simple_gripper.xacro"/>
     <!-- Import ros2_control macros -->
     <xacro:include filename="$(find kawada_moveit_config)/config/NEXTAGE.ros2_control.xacro"/>
@@ -29,3 +31,7 @@
         name="LeftArmSystem"
         initial_positions_file="$(arg initial_positions_file)"/>
+    <!-- Add gripper to right arm end-effector -->
+    <xacro:simple_gripper prefix="right" parent="RARM_JOINT5_Link">
+        <origin xyz="0 0 -0.05" rpy="0 0 0"/>
+    </xacro:simple_gripper>
 </robot>

File: kawada_repo-main/nextage_fillie_open_description/urdf/nextage_fillie_open_gz.xacro (robot description, xacro)
@@ -29,5 +29,3 @@
          link_displacement_x="0.0325" link_displacement_y="0" link_displacement_z="0"
          link_rotation_x="0" link_rotation_y="${M_PI/2}" link_rotation_z="${link_head_camera_rot_z}" /> -->
-  <!-- TODO hand cameras can be added here with the very similar code as
-            headmount cameras. -->
 </robot>

Commit message: Add dual-arm Robotiq grippers
- Replace simple gripper with Robotiq 2F-140 style grippers
- Add grippers to both left and right arms
- Configure ROS2 controllers for both grippers

File: kawada_repo-main/kawada_moveit_config/config/NEXTAGE.ros2_control.xacro (robot description, xacro)
@@ -50,5 +50,5 @@
                 <state_interface name="velocity"/>
             </joint>
-            <joint name="right_gripper_left_finger_joint">
+            <joint name="right_left_finger_joint">
                 <command_interface name="position"/>
                 <state_interface name="position">
@@ -56,4 +56,13 @@
                 </state_interface>
                 <state_interface name="velocity"/>
+                <state_interface name="effort"/>
+            </joint>
+            <joint name="left_left_finger_joint">
+                <command_interface name="position"/>
+                <state_interface name="position">
+                  <param name="initial_value">0.0</param>
+                </state_interface>
+                <state_interface name="velocity"/>
+                <state_interface name="effort"/>
             </joint>
         </ros2_control>

File: kawada_repo-main/kawada_moveit_config/config/NEXTAGE.urdf.xacro (robot description, xacro)
@@ -19,6 +19,6 @@
     <!-- Import cameras -->
     <xacro:include filename="$(find kawada_moveit_config)/config/cameras.xacro"/>
-    <!-- Import gripper -->
-    <xacro:include filename="$(find nextage_fillie_open_description)/urdf/simple_gripper.xacro"/>
+    <!-- Import new gripper -->
+    <xacro:include filename="$(find nextage_fillie_open_description)/urdf/robotiq_2f_140_gripper.xacro"/>
     <!-- Import ros2_control macros -->
     <xacro:include filename="$(find kawada_moveit_config)/config/NEXTAGE.ros2_control.xacro"/>
@@ -31,7 +31,10 @@
         name="LeftArmSystem"
         initial_positions_file="$(arg initial_positions_file)"/>
-    <!-- Add gripper to right arm end-effector -->
-    <xacro:simple_gripper prefix="right" parent="RARM_JOINT5_Link">
-        <origin xyz="0 0 -0.05" rpy="0 0 0"/>
-    </xacro:simple_gripper>
+    <!-- Add grippers to both arms -->
+    <xacro:robotiq_gripper prefix="right" parent="RARM_JOINT5_Link">
+        <origin xyz="0 0 0" rpy="0 0 0"/>
+    </xacro:robotiq_gripper>
+    <xacro:robotiq_gripper prefix="left" parent="LARM_JOINT5_Link">
+        <origin xyz="0 0 0" rpy="0 0 0"/>
+    </xacro:robotiq_gripper>
 </robot>

File: kawada_repo-main/nextage_fillie_open_description/urdf/FillieOpen.urdf (robot description, URDF)
Before this commit: robot NEXTAGE, 16 links, 15 joints
Joints:
- joint RARM_JOINT0: limit lower=-1.570796327 upper=1.570796327 effort=150 velocity=1.0 -> lower=-1.570796327 upper=1.570796327 effort=150 velocity=100.0
- joint RARM_JOINT1: limit lower=-2.443460953 upper=1.570796327 effort=150 velocity=1.0 -> lower=-2.443460953 upper=1.570796327 effort=150 velocity=100.0
- joint RARM_JOINT2: limit lower=-1.221730476 upper=1.570796327 effort=150 velocity=1.0 -> lower=-1.221730476 upper=1.570796327 effort=150 velocity=100.0
- joint RARM_JOINT3: limit lower=-1.745329252 upper=3.141592654 effort=150 velocity=1.0 -> lower=-1.745329252 upper=3.141592654 effort=150 velocity=100.0
- joint RARM_JOINT4: limit lower=-1.570796327 upper=1.570796327 effort=150 velocity=1.0 -> lower=-1.570796327 upper=1.570796327 effort=150 velocity=100.0
- joint RARM_JOINT5: limit lower=-2.9670597283903604 upper=2.9670597283903604 effort=150 velocity=1.0 -> lower=-2.9670597283903604 upper=2.9670597283903604 effort=150 velocity=100.0

File: kawada_repo-main/nextage_fillie_open_description/urdf/nextage_fillie_open_gz.xacro (robot description, xacro)
@@ -4,4 +4,5 @@
   <xacro:include filename="$(find nextage_fillie_open_description)/urdf/FillieOpen.urdf" />
   <xacro:include filename="$(find nextage_fillie_open_description)/urdf/nextage_fillie_open_gz_camera.xacro" />
+  <xacro:include filename="$(find nextage_fillie_open_description)/urdf/robotiq_2f_140_gripper.xacro" />
   <!-- <xacro:property name="M_PI" value="3.1415926535897931" />
   <xacro:property name="jnt_head_camera_displacement_x" value="0.0175" />
@@ -29,3 +30,11 @@
          link_displacement_x="0.0325" link_displacement_y="0" link_displacement_z="0"
          link_rotation_x="0" link_rotation_y="${M_PI/2}" link_rotation_z="${link_head_camera_rot_z}" /> -->
+  <!-- Add Robotiq 2F-140 Gripper to right arm -->
+  <xacro:robotiq_gripper prefix="right" parent="RARM_JOINT5_Link">
+    <origin xyz="0.0 0.0 0.0" rpy="0 0 0"/>
+  </xacro:robotiq_gripper>
+  <!-- Add Robotiq 2F-140 Gripper to left arm -->
+  <xacro:robotiq_gripper prefix="left" parent="LARM_JOINT5_Link">
+    <origin xyz="0.0 0.0 0.0" rpy="0 0 0"/>
+  </xacro:robotiq_gripper>
 </robot>
